File: CanSwitch2.kicad_pcb (KiCad board)
At the start: 2 copper layers, 25.4 x 50.8 mm, 5 parts, among them J1 250-202 Wago, J2 250-202 Wago, SW1 SW_Slide_DPDT

Commit message: CJ's Update
Connections:
- R1 pad 1: Net-(J1-Pad1) -> Net-(J1-Pad2)
- R2 pad 2: Net-(J2-Pad1) -> Net-(J2-Pad2)
Routing:
- net Net-(J1-Pad2): track 10.5 -> 33.6 mm
- net Net-(J2-Pad2): track 16.6 -> 28.0 mm
- net Net-(J1-Pad1): track 21.2 -> 14.5 mm
- net Net-(J2-Pad1): track 19.9 -> 14.3 mm
Changed lines of the file:
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@@
 			(layers "F.Cu" "F.Paste" "F.Mask")
 			(roundrect_rratio 0.243902)
-			(net 2 "Net-(J1-Pad1)")
+			(net 1 "Net-(J1-Pad2)")
 			(pintype "passive")
 		)
@@
 			(layers "F.Cu" "F.Paste" "F.Mask")
 			(roundrect_rratio 0.243902)
-			(net 6 "Net-(J2-Pad1)")
+			(net 3 "Net-(J2-Pad2)")
 			(pintype "passive")
 		)
@@
 	)
 	(gr_text "Terminate"
-		(at 22 42 90)
+		(at 23.5 42 90)
 		(layer "F.SilkS")
 		(effects
@@
 	)
 	(gr_text "Passthru"
-		(at 22.5 23.5 90)
+		(at 24 23.5 90)
 		(layer "F.SilkS")
 		(effects
@@
 	)
 	(segment
+		(start 13.875 11.875)
+		(end 15 13)
+		(width 0.2)
+		(layer "F.Cu")
+		(net 1)
+	)
+	(segment
+		(start 15 23.4882)
+		(end 15.0118 23.5)
+		(width 0.2)
+		(layer "F.Cu")
+		(net 1)
+	)
+	(segment
 		(start 15 18.5)
 		(end 15 13)
@@
 	)
 	(segment
-		(start 15 23.4882)
-		(end 15.0118 23.5)
+		(start 9.534009 11.875)
+		(end 13.875 11.875)
 		(width 0.2)
 		(layer "F.Cu")
@@
 	)
 	(segment
-		(start 5.0118 23.4882)
-		(end 5.0118 27.175)
+		(start 5.0118 27.175)
+		(end 5.0118 16.397209)
+		(width 0.2)
+		(layer "F.Cu")
+		(net 1)
+	)
+	(segment
+		(start 5.0118 16.397209)
+		(end 9.534009 11.875)
+		(width 0.2)
+		(layer "F.Cu")
+		(net 1)
+	)
+	(segment
+		(start 7.9554 20.5446)
+		(end 7.9554 24.4554)
 		(width 0.2)
 		(layer "F.Cu")
@@
 	(segment
 		(start 10 18.5)
-		(end 5.0118 23.4882)
+		(end 7.9554 20.5446)
 		(width 0.2)
 		(layer "F.Cu")
@@
 	)
 	(segment
-		(start 9.5 26)
-		(end 6.1868 26)
-		(width 0.2)
-		(layer "F.Cu")
-		(net 2)
-	)
-	(segment
-		(start 6.1868 26)
-		(end 5.0118 27.175)
+		(start 7.9554 24.4554)
+		(end 9.5 26)
 		(width 0.2)
 		(layer "F.Cu")
@@
 	)
 	(segment
+		(start 19.5118 26.675)
+		(end 17.8814 25.0446)
+		(width 0.2)
+		(layer "F.Cu")
+		(net 3)
+	)
+	(segment
+		(start 11.0446 32.4554)
+		(end 11.0446 25.0446)
+		(width 0.2)
+		(layer "F.Cu")
+		(net 3)
+	)
+	(segment
 		(start 10 33.5)
 		(end 11.0446 32.4554)
@@
 	)
 	(segment
+		(start 9.5 23.5)
+		(end 11.1031 25.1031)
+		(width 0.2)
+		(layer "F.Cu")
+		(net 3)
+	)
+	(segment
+		(start 17.8814 25.0446)
+		(end 11.0446 25.0446)
+		(width 0.2)
+		(layer "F.Cu")
+		(net 3)
+	)
+	(segment
 		(start 11.0446 25.0446)
 		(end 9.5 23.5)
@@
 	)
 	(segment
-		(start 11.0446 32.4554)
-		(end 11.0446 25.0446)
-		(width 0.2)
-		(layer "F.Cu")
-		(net 3)
-	)
-	(segment
 		(start 10 33.5)
 		(end 10 39)
@@
 	)
 	(segment
-		(start 5.0118 29)
+		(start 9.5 28.5)
 		(end 9 29)
 		(width 0.2)
@@
 	(segment
 		(start 9 29)
-		(end 9.5 28.5)
+		(end 5.0118 29)
 		(width 0.2)
 		(layer "F.Cu")
@@
 	(segment
 		(start 15 33.5)
-		(end 12.5 31)
+		(end 13.4672 31.9672)
 		(width 0.2)
 		(layer "F.Cu")
@@
 	)
 	(segment
-		(start 15.0118 26)
-		(end 18.8368 26)
+		(start 13.4672 27.5446)
+		(end 15.0118 26)
 		(width 0.2)
 		(layer "F.Cu")
@@
 	)
 	(segment
-		(start 18.8368 26)
-		(end 19.5118 26.675)
-		(width 0.2)
-		(layer "F.Cu")
-		(net 6)
-	)
-	(segment
-		(start 12.5 28.5118)
-		(end 15.0118 26)
+		(start 13.4672 31.9672)
+		(end 13.4672 27.5446)
 		(width 0.2)
 		(layer "F.Cu")
@@
 		(width 0.2)
 		(layer "F.Cu")
-		(net 6)
-	)
-	(segment
-		(start 12.5 31)
-		(end 12.5 28.5118)
-		(width 0.2)
-		(layer "F.Cu")
