File: CanSwitch2.kicad_sch (KiCad schematic)
At the start: 5 parts, among them J1 250-202 Wago, J2 250-202 Wago, SW1 SW_Slide_DPDT

Commit message: CJ's Update
Connections:
- net at J1.1, J1.4, SW1.2 (B): no longer R1.1
- net at J1.2, J1.3, SW1.6 (C): now also R1.1
- net at J2.1, J2.4, SW1.5 (B): no longer R2.2
- net at J2.2, J2.3, SW1.1 (A): now also R2.2
Other:
- moved on the sheet: J2
Changed lines of the file:
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@@
 	(paper "A4")
-	(junction
-		(at 100.33 142.24)
-		(diameter 0)
-		(color 0 0 0 0)
-	)
 	(junction
 		(at 101.6 53.34)
@@
 	)
 	(junction
+		(at 82.55 110.49)
+		(diameter 0)
+		(color 0 0 0 0)
+	)
+	(junction
 		(at 101.6 55.88)
 		(diameter 0)
@@
 	)
 	(junction
-		(at 64.77 92.71)
-		(diameter 0)
-		(color 0 0 0 0)
-	)
-	(junction
 		(at 102.87 121.92)
 		(diameter 0)
@@
 	)
 	(junction
-		(at 125.73 97.79)
+		(at 82.55 119.38)
 		(diameter 0)
 		(color 0 0 0 0)
 	)
-	(junction
-		(at 125.73 119.38)
-		(diameter 0)
-		(color 0 0 0 0)
-	)
-	(wire
-		(pts
-			(xy 125.73 97.79) (xy 125.73 119.38)
-		)
-		(stroke
-			(width 0)
-			(type default)
-		)
-	)
-	(wire
-		(pts
-			(xy 104.14 72.39) (xy 119.38 72.39)
-		)
-		(stroke
-			(width 0)
-			(type default)
-		)
-	)
-	(wire
-		(pts
-			(xy 100.33 142.24) (xy 102.87 142.24)
+	(wire
+		(pts
+			(xy 82.55 110.49) (xy 82.55 119.38)
 		)
 		(stroke
@@
 	(wire
 		(pts
-			(xy 64.77 97.79) (xy 64.77 92.71)
-		)
-		(stroke
-			(width 0)
-			(type default)
-		)
-	)
-	(wire
-		(pts
 			(xy 121.92 53.34) (xy 121.92 55.88)
 		)
@@
 	(wire
 		(pts
-			(xy 125.73 97.79) (xy 125.73 92.71)
+			(xy 125.73 92.71) (xy 125.73 119.38)
 		)
 		(stroke
@@
 	(wire
 		(pts
-			(xy 41.91 92.71) (xy 64.77 92.71)
-		)
-		(stroke
-			(width 0)
-			(type default)
-		)
-	)
-	(wire
-		(pts
 			(xy 119.38 87.63) (xy 105.41 87.63)
 		)
@@
 	(wire
 		(pts
-			(xy 82.55 146.05) (xy 100.33 146.05)
-		)
-		(stroke
-			(width 0)
-			(type default)
-		)
-	)
-	(wire
-		(pts
-			(xy 125.73 119.38) (xy 125.73 153.67)
-		)
-		(stroke
-			(width 0)
-			(type default)
-		)
-	)
-	(wire
-		(pts
-			(xy 82.55 87.63) (xy 82.55 146.05)
+			(xy 82.55 87.63) (xy 82.55 110.49)
 		)
 		(stroke
@@
 	(wire
 		(pts
+			(xy 82.55 119.38) (xy 82.55 121.92)
+		)
+		(stroke
+			(width 0)
+			(type default)
+		)
+	)
+	(wire
+		(pts
 			(xy 101.6 33.02) (xy 104.14 33.02)
 		)
@@
 	(wire
 		(pts
-			(xy 64.77 92.71) (xy 95.25 92.71)
+			(xy 86.36 97.79) (xy 86.36 72.39)
+		)
+		(stroke
+			(width 0)
+			(type default)
+		)
+	)
+	(wire
+		(pts
+			(xy 41.91 92.71) (xy 95.25 92.71)
 		)
 		(stroke
@@
 	(wire
 		(pts
-			(xy 118.11 97.79) (xy 125.73 97.79)
-		)
-		(stroke
-			(width 0)
-			(type default)
-		)
-	)
-	(wire
-		(pts
 			(xy 101.6 53.34) (xy 101.6 55.88)
 		)
@@
 	(wire
 		(pts
+			(xy 118.11 97.79) (xy 118.11 110.49)
+		)
+		(stroke
+			(width 0)
+			(type default)
+		)
+	)
+	(wire
+		(pts
 			(xy 101.6 60.96) (xy 101.6 55.88)
 		)
@@
 	(wire
 		(pts
-			(xy 100.33 146.05) (xy 100.33 142.24)
-		)
-		(stroke
-			(width 0)
-			(type default)
-		)
-	)
-	(wire
-		(pts
 			(xy 119.38 72.39) (xy 119.38 87.63)
 		)
@@
 	(wire
 		(pts
+			(xy 118.11 110.49) (xy 82.55 110.49)
+		)
+		(stroke
+			(width 0)
+			(type default)
+		)
+	)
+	(wire
+		(pts
 			(xy 100.33 121.92) (xy 102.87 121.92)
 		)
@@
 	(wire
 		(pts
-			(xy 64.77 97.79) (xy 86.36 97.79)
+			(xy 86.36 72.39) (xy 119.38 72.39)
 		)
 		(stroke
@@
 	(symbol
 		(lib_id "Weidmuller:1825960000 2pos wide")
-		(at 102.87 121.92 270)
+		(at 102.87 121.92 180)
 		(unit 1)
 		(exclude_from_sim no)
@@
 		(fields_autoplaced yes)
 		(property "Reference" "J2"
-			(at 106.68 130.8099 90)
+			(at 93.9801 125.73 90)
 			(effects
 				(font
@@
 		)
 		(property "Value" "250-202 Wago"
-			(at 106.68 133.3499 90)
+			(at 91.4401 125.73 90)
 			(effects
 				(font
@@
 		)
 		(property "Footprint" "1825960000"
-			(at 7.95 138.43 0)
+			(at 86.36 27 0)
 			(effects
 				(font
@@
 		)
 		(property "Datasheet" "http://catalog.weidmueller.com/createDatasheetForMobile.do?ordernumber=1825960000&scope1=1&scope2=1&localeId=en"
-			(at -92.05 138.43 0)
+			(at 86.36 -73 0)
 			(effects
 				(font
@@
 		)
 		(property "Height" "14"
-			(at -292.05 138.43 0)
+			(at 86.36 -273 0)
 			(effects
 				(font
@@
 		)
 		(property "Manufacturer_Name" "Weidmuller"
-			(at -392.05 138.43 0)
+			(at 86.36 -373 0)
 			(effects
 				(font
@@
 		)
 		(property "Manufacturer_Part_Number" "1825960000"
-			(at -492.05 138.43 0)
+			(at 86.36 -473 0)
 			(effects
 				(font
@@
 		)
 		(property "Mouser Part Number" "470-1825960000"
-			(at -592.05 138.43 0)
+			(at 86.36 -573 0)
 			(effects
 				(font
@@
 		)
 		(property "Mouser Price/Stock" "https://www.mouser.co.uk/ProductDetail/Weidmuller/1825960000?qs=BTG2th8YmhTHqEF9wcCIDA%3D%3D"
-			(at -692.05 138.43 0)
+			(at 86.36 -673 0)
 			(effects
 				(font
@@
 		)
 		(property "Arrow Part Number" ""
-			(at -792.05 138.43 0)
+			(at 86.36 -773 0)
 			(effects
 				(font
@@
 		)
 		(property "Arrow Price/Stock" ""
-			(at -892.05 138.43 0)
-			(effects
-				(font
+			(at 86.36 -873 0)
+			(effects
+				(font
